Commit message: bugfixes from practice

File: kc_vision/urdf/mk2_robot.urdf (robot description, URDF)
Before this commit: robot mk2, 2 links, 1 joints
Links:
- added link robot
- link front_camera: geometry visual box size=0.08 0.04 0.02
Joints:
- added joint robot_to_chassis: type fixed, parent robot, child chassis
- joint chassis_to_front_camera: origin xyz=0.5 0 0.5 rpy=-1.57079 0 -1.57079 -> xyz=0 0 0.5

Commit message: restructured intake camera node

File: kc_vision/urdf/mk2_robot.urdf (robot description, URDF)
Before this commit: robot mk2, 3 links, 2 joints
Links:
- added link intake_camera; visual box size=0.08 0.04 0.02
Joints:
- added joint chassis_to_intake_camera: type fixed, parent chassis, child intake_camera, origin xyz=0 0.1 0.5 rpy=-1.57079 0 -1.57079

Commit message: switched to using depthai ros driver and began implementation of detection_location_calculator

File: kc_vision/urdf/mk2_robot.urdf (robot description, URDF)
Before this commit: robot mk2, 4 links, 3 joints
Joints:
- joint chassis_to_intake_camera: origin xyz=0 0.1 0.5 rpy=-1.57079 0 -1.57079 -> xyz=0 0.1 0.5
