Commit message: grid fuel detector debugging

File: kc_vision/urdf/mk1_robot.urdf (robot description, URDF)
Before this commit: robot mk2, 6 links, 5 joints
Joints:
- removed joint robot_to_front_grid
- added joint front_camera_to_front_grid: type fixed, parent front_camera, child front_grid, origin xyz=0 0 1 rpy=3.14159 0 -1.5708

Commit message: changes for full integration testing

File: kc_vision/urdf/mk1_robot.urdf (robot description, URDF)
Before this commit: robot mk2, 6 links, 5 joints
Links:
- removed link front_grid
- added link front_camera_interstitial
- added link intake_camera_interstitial
- added link intake_grid
Joints:
- removed joint front_camera_to_front_grid
- removed joint robot_to_front_camera
- removed joint robot_to_intake_camera
- added joint front_camera_interstitial_to_front_camera: type fixed, parent front_camera_interstitial, child front_camera, origin rpy=0 0 -1.5708
- added joint intake_camera_interstitial_to_intake_camera: type fixed, parent intake_camera_interstitial, child intake_camera, origin rpy=0 0 -1.5708
- added joint robot_to_front_camera_interstitial: type fixed, parent robot, child front_camera_interstitial, origin xyz=0.263630 -0.175331 0.687403 rpy=-1.396263 0 -1.5708
- added joint robot_to_intake_camera_interstitial: type fixed, parent robot, child intake_camera, origin xyz=0.251043 0.002469 0.682677 rpy=-1.832596 0 -1.5708
- added joint robot_to_intake_grid: type fixed, parent robot, child intake_grid, origin xyz=1 0 0.1

Commit message: mostly functioning apriltag localization

File: kc_vision/urdf/mk1_robot.urdf (robot description, URDF)
Before this commit: robot v1, 8 links, 7 joints
Joints:
- joint robot_to_intake_camera_interstitial: child intake_camera -> intake_camera_interstitial
- joint robot_to_intake_grid: origin xyz=1 0 0.1 -> xyz=0.89 -0.3429 0.1

Commit message: working vision with Isaac ROS acceleration

File: kc_vision/urdf/mk1_robot.urdf (robot description, URDF)
Before this commit: robot v1, 8 links, 7 joints
Links:
- added link oak
- added link oak_interstitial
Joints:
- added joint oak_interstitial_to_oak: type fixed, parent oak_interstitial, child oak, origin rpy=3.14159 0 0
- added joint robot_to_oak_interstitial: type fixed, parent robot, child oak_interstitial, origin xyz=0.252628 0.120650 0.708825 rpy=0 0.261799 0
