Commit message: Fuel data over NT, and added right camera april tag tracking

File: kc_vision/urdf/mk1_robot.urdf (robot description, URDF)
Before this commit: robot v1, 10 links, 9 joints
Links:
- removed link back_right_camera
- added link right_camera; visual box size=0.05715 0.05715 0.02
Joints:
- removed joint robot_to_back_right_camera
- added joint robot_to_right_camera: type fixed, parent robot, child right_camera, origin xyz=0.145311 -0.303003 0.708814 rpy=-1.184 -0.363 2.288
- joint robot_to_intake_grid: origin xyz=0.89 -0.3429 0.1 -> xyz=0.89 -0.6858 0.1

File: kc_vision/urdf/mk2_robot.urdf (robot description, URDF)
Before this commit: robot mk2, 4 links, 3 joints
Links:
- added link right_camera; visual box size=0.08 0.04 0.02
Joints:
- added joint chassis_to_right_camera: type fixed, parent chassis, child right_camera, origin xyz=0.145311 -0.303003 0.708814 rpy=-1.5708 0 3.14159
- joint chassis_to_front_camera: origin xyz=0 0 0.5 -> xyz=0 0.1 0.5
